File: eagle/v0.91/ESP32K40.brd (EAGLE design)
At the start: 97 x 64 mm, 21 parts, among them J1 uSTEPX, J2 uSTEPY, K40FFC 1-84534-2, Q2 2N7002

Commit message: proper mosfet type
Parts:
- Q2: value 2N7002 -> p75nf75
Changed lines of the file:
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@@
 <attribute name="VALUE" x="66.964" y="-1.0466" size="1.27" layer="27"/>
 </element>
-<element name="Q2" library="adafruit" library_urn="urn:adsk.eagle:library:420" package="TO220V" package3d_urn="urn:adsk.eagle:package:6240882/1" value="2N7002" x="49.53" y="9.779" smashed="yes">
+<element name="Q2" library="adafruit" library_urn="urn:adsk.eagle:library:420" package="TO220V" package3d_urn="urn:adsk.eagle:package:6240882/1" value="p75nf75" x="49.53" y="9.779" smashed="yes">
 <attribute name="NAME" x="55.88" y="7.5438" size="1.27" layer="25" ratio="10"/>
 <attribute name="VALUE" x="46.99" y="9.779" size="1.27" layer="27" ratio="10"/>
